File: rio-iceshield.kicad_pcb (KiCad board)
At the start: 2 copper layers, 87.6 x 56 mm, 94 parts, among them J2 Conn_01x06, J3 Conn_01x06, J4 Conn_01x06, J5 Conn_01x06, J6 Conn_01x06, J7 Conn_02x06_Odd_Even, U1 ICE40UP5K-SG48ITR, U10 PC817, U11 PC817, U12 PC817, U13 PC817, U14 PC817, U2 AT25SF041B-SHD 4 Mb, U3 LD3985M122R_SOT23, U4 ULN2803A, U5 ULN2803A, U7 PC817, U8 PC817, U9 PC817, X2 XO91, j1 GPIO

Commit message: update
Parts:
- removed MH1, MH2, MH3, MH4: MountingHole_2.7mm_M2.5, MountingHole:MountingHole_2.7mm_M2.5
- added REF**: MountingHole_3.2mm_M3, MountingHole:MountingHole_3.2mm_M3, F.Cu at (103.5, 96.5)
- added REF**: MountingHole_3.2mm_M3, MountingHole:MountingHole_3.2mm_M3, F.Cu at (161.5, 47.5)
- added REF**: MountingHole_3.2mm_M3, MountingHole:MountingHole_3.2mm_M3, F.Cu at (161.5, 96.5)
- added REF**: MountingHole_3.2mm_M3, MountingHole:MountingHole_3.2mm_M3, F.Cu at (103.5, 47.5)
- renumbered +24V-1 to +24V
Routing:
- net gnd: vias 19 -> 18
Other:
- board text added: "R2"
- board text added: "R28"
- board text added: "R29"
- board text added: "R3"
- board text added: "R30"
- board text added: "R4"
- board text added: "U10"
- board text added: "U11"
- board text added: "U12"
- board text added: "U13"
- board text added: "U14"
- board text added: "U3"
- board text added: "U4"
- board text added: "U7"
- board text added: "U8"
- board text added: "U9"
